Commit message: changes for working visualisation based on different postion input

File: ros_ws/src/prototype_description/urdf/my_bot.ros2_control.xacro (robot description, xacro)
@@ -14,4 +14,12 @@
             <state_interface name="position" />
         </joint>
+        <joint name="Revolute_3">
+            <command_interface name="position" />
+            <state_interface name="position" />
+        </joint>
+        <joint name="Revolute_4">
+            <command_interface name="position" />
+            <state_interface name="position" />
+        </joint>
         <joint name="Revolute_5">
             <command_interface name="position" />
@@ -22,4 +30,12 @@
             <state_interface name="position" />
         </joint>
+        <joint name="Revolute_7">
+            <command_interface name="position" />
+            <state_interface name="position" />
+        </joint>
+        <joint name="Revolute_8">
+            <command_interface name="position" />
+            <state_interface name="position" />
+        </joint>
     </ros2_control>
 </robot>

File: ros_ws/src/prototype_description/urdf/my_bot_urdf.xacro (robot description, xacro)
@@ -196,6 +196,6 @@
   <parent link="Chassis_Right_1"/>
   <child link="backLeg_Right_1"/>
-  <axis xyz="0.0 1.0 -0.0"/>
-  <limit upper="0.349066" lower="-1.919862" effort="100" velocity="100"/>
+  <axis xyz="-0.0 -1.0 0.0"/>
+  <limit upper="1.919862" lower="-0.349066" effort="100" velocity="100"/>
 </joint>
 <joint name="Revolute_3" type="continuous">
@@ -215,6 +215,6 @@
   <parent link="base_link"/>
   <child link="Chassis_Left_1"/>
-  <axis xyz="0.0 1.0 -0.0"/>
-  <limit upper="1.396263" lower="-0.698132" effort="100" velocity="100"/>
+  <axis xyz="-0.0 -1.0 0.0"/>
+  <limit upper="0.698132" lower="-1.396263" effort="100" velocity="100"/>
 </joint>
 <joint name="Revolute_6" type="revolute">
